Commit message: Added calibration attachment to robot base.

File: franka_description/robots/common/franka_arm.xacro (robot description, xacro)
@@ -18,4 +18,14 @@
       </self_collision_geometries>
     </xacro:link_with_sc>
+    <xacro:link_with_sc name="link_base_calibration_attachment" gazebo="${gazebo}">
+      <self_collision_geometries>
+        <xacro:collision_capsule xyz="0.0 0.0 0.0" direction="x" radius="${0.01+safety_distance}" length="0.01" />
+      </self_collision_geometries>
+    </xacro:link_with_sc>
+    <joint name="${arm_id}_joint_base_calibration_attachment" type="fixed">
+      <parent link="${arm_id}_link0"/>
+      <child link="${arm_id}_link_base_calibration_attachment"/>
+      <origin rpy="0 0 -1.57079632679" xyz="-0.015 0.1086 -0.021" />
+    </joint>
     <xacro:link_with_sc name="link1" gazebo="${gazebo}">
       <self_collision_geometries>

Commit message: Fixed collisions and measurement error

File: franka_description/robots/common/franka_arm.xacro (robot description, xacro)
@@ -20,5 +20,5 @@
     <xacro:link_with_sc name="link_base_calibration_attachment" gazebo="${gazebo}">
       <self_collision_geometries>
-        <xacro:collision_capsule xyz="0.0 0.0 0.0" direction="x" radius="${0.01+safety_distance}" length="0.01" />
+        <xacro:collision_capsule xyz="0.0 0.0 0.0" direction="x" radius="${0.001}" length="0.001" />
       </self_collision_geometries>
     </xacro:link_with_sc>
@@ -26,5 +26,5 @@
       <parent link="${arm_id}_link0"/>
       <child link="${arm_id}_link_base_calibration_attachment"/>
-      <origin rpy="0 0 -1.57079632679" xyz="-0.015 0.1086 -0.021" />
+      <origin rpy="0 0 -1.57079632679" xyz="-0.015 0.1086 -0.02" />
     </joint>
     <xacro:link_with_sc name="link1" gazebo="${gazebo}">
