Commit message: Changed pump related link names to use the word pump instead of hand, and adjusted pump tcp position (previously was copied exactly from hand tcp position).

File: franka_description/robots/common/franka_pump.xacro (robot description, xacro)
@@ -1,10 +1,10 @@
 <?xml version="1.0" encoding="utf-8"?>
-<robot xmlns:xacro="http://www.ros.org/wiki/xacro" name="hand">
+<robot xmlns:xacro="http://www.ros.org/wiki/xacro" name="pump">
   <!-- safety_distance: Minimum safety distance in [m] by which the collision volumes are expanded and which is enforced during robot motions -->
   <xacro:macro name="franka_pump" params="connected_to:='' arm_id:='panda' rpy:='0 0 0' xyz:='0 0 0' tcp_xyz:='0 0 0.1034' tcp_rpy:='0 0 0' safety_distance:=0 gazebo:=false description_pkg:=franka_description">
     <xacro:unless value="${connected_to == ''}">
-      <joint name="${arm_id}_hand_joint" type="fixed">
+      <joint name="${arm_id}_pump_joint" type="fixed">
         <parent link="${connected_to}" />
-        <child link="${arm_id}_hand" />
+        <child link="${arm_id}_pump" />
         <origin xyz="${xyz}" rpy="${rpy}" />
       </joint>
@@ -16,5 +16,5 @@
       </self_collision_geometries>
     </xacro:link_with_sc> -->
-    <link name="${arm_id}_hand" >
+    <link name="${arm_id}_pump" >
       <visual>
         <origin xyz="0 0 0" rpy="0 ${pi} 0"/>
@@ -40,9 +40,9 @@
     </joint> -->
     <!-- Define the hand_tcp frame -->
-    <link name="${arm_id}_hand_tcp" />
-    <joint name="${arm_id}_hand_tcp_joint" type="fixed">
+    <link name="${arm_id}_pump_tcp" />
+    <joint name="${arm_id}_pump_tcp_joint" type="fixed">
       <origin xyz="${tcp_xyz}" rpy="${tcp_rpy}" />
-      <parent link="${arm_id}_hand" />
-      <child link="${arm_id}_hand_tcp" />
+      <parent link="${arm_id}_pump" />
+      <child link="${arm_id}_pump_tcp" />
     </joint>
     <!-- <link name="${arm_id}_pump">

File: franka_description/robots/common/franka_robot.xacro (robot description, xacro)
@@ -11,4 +11,8 @@
     <!-- Rotational offset between $(arm_id)_hand -> $(arm_id)_hand_tcp [rad]. Only used when hand:=true -->
     <xacro:arg name="tcp_rpy" default="0 0 0" />
+    <!-- Positional offset between $(arm_id)_pump -> $(arm_id)_pump_tcp [m]. Only used when pump:=true -->
+    <xacro:arg name="pump_tcp_xyz" default="0 0 0.115" />
+    <!-- Rotational offset between $(arm_id)_pump -> $(arm_id)_pump_tcp [rad]. Only used when pump:=true -->
+    <xacro:arg name="pump_tcp_rpy" default="0 0 0" />
     <!-- Is the robot being simulated in gazebo?" -->
     <xacro:arg name="gazebo" default="false" />
@@ -33,6 +37,6 @@
           arm_id="$(arg arm_id)"
           rpy="0 0 ${-pi/4}"
-          tcp_xyz="$(arg tcp_xyz)"
-          tcp_rpy="$(arg tcp_rpy)"
+          tcp_xyz="$(arg pump_tcp_xyz)"
+          tcp_rpy="$(arg pump_tcp_rpy)"
           connected_to="$(arg arm_id)_link8"
           safety_distance="0.03"

Commit message: Removed commented out model code from pump xacro. Addied long pump xacro based off pump xacro with additional cylinder visual and collision mesh. Modified franka_robot so that it an load long pump xacro based off arguments. Added argument to high level panda.launch file.

File: franka_description/robots/common/franka_pump.xacro (robot description, xacro)
@@ -10,10 +10,4 @@
       </joint>
     </xacro:unless>
-    <!-- <xacro:link_with_sc name="pump_simplified" gazebo="${gazebo}">
-      <self_collision_geometries>
-        <xacro:collision_capsule xyz="0 0 0.04" direction="y" radius="${0.04+safety_distance}" length="0.1" />
-        <xacro:collision_capsule xyz="0 0 0.10" direction="y" radius="${0.02+safety_distance}" length="0.1" />
-      </self_collision_geometries>
-    </xacro:link_with_sc> -->
     <link name="${arm_id}_pump" >
       <visual>
@@ -33,10 +27,4 @@
       </xacro:if>
     </link>
-    <!-- <joint name="${arm_id}_hand" type="fixed">
-      <parent link="${arm_id}_link8" />
-      <child link="${arm_id}_hand" />
-      <origin xyz="0 0 0.0584" rpy="0 0 0" />
-      <axis xyz="0 1 0" />
-    </joint> -->
     <!-- Define the hand_tcp frame -->
     <link name="${arm_id}_pump_tcp" />
@@ -46,23 +34,4 @@
       <child link="${arm_id}_pump_tcp" />
     </joint>
-    <!-- <link name="${arm_id}_pump">
-      <visual>
-        <geometry>
-          <mesh filename="package://${description_pkg}/meshes/visual/pump_simplified.dae" />
-        </geometry>
-      </visual>
-      <collision>
-        <origin xyz="0 0 0.05" rpy="0 0 ${pi/2}"/>
-        <geometry>
-          <cylinder radius="${0.05+safety_distance}" length="0.12" />
-        </geometry>
-      </collision>
-    </link>
-    <joint name="${arm_id}_finger_joint1" type="fixed">
-      <parent link="${arm_id}_hand" />
-      <child link="${arm_id}_pump" />
-      <origin xyz="0 0 0.0584" rpy="0 0 0" />
-      <axis xyz="0 1 0" />
-    </joint> -->
   </xacro:macro>
 </robot>

File: franka_description/robots/common/franka_robot.xacro (robot description, xacro)
@@ -7,4 +7,6 @@
     <!-- Should a franka_pump be mounted at the flange?" -->
     <xacro:arg name="pump" default="false" />
+    <!-- Should a franka_pump with a long rod be mounted at the flange?" -->
+    <xacro:arg name="long_pump" default="false" />
     <!-- Positional offset between $(arm_id)_hand -> $(arm_id)_hand_tcp [m]. Only used when hand:=true -->
     <xacro:arg name="tcp_xyz" default="0 0 0.1034" />
@@ -15,4 +17,8 @@
     <!-- Rotational offset between $(arm_id)_pump -> $(arm_id)_pump_tcp [rad]. Only used when pump:=true -->
     <xacro:arg name="pump_tcp_rpy" default="0 0 0" />
+    <!-- Positional offset between $(arm_id)_long_pump -> $(arm_id)_pump_tcp [m]. Only used when pump:=true -->
+    <xacro:arg name="long_pump_tcp_xyz" default="0 0 0.34" /> <!-- TOO - check thils tcp offset for long pump -->
+    <!-- Rotational offset between $(arm_id)_long_pump -> $(arm_id)_pump_tcp [rad]. Only used when pump:=true -->
+    <xacro:arg name="long_pump_tcp_rpy" default="0 0 0" />
     <!-- Is the robot being simulated in gazebo?" -->
     <xacro:arg name="gazebo" default="false" />
@@ -20,4 +26,5 @@
     <xacro:include filename="$(find franka_description)/robots/common/franka_arm.xacro" />
     <xacro:franka_arm arm_id="${arm_id}" safety_distance="0.03" gazebo="$(arg gazebo)" joint_limits="${joint_limits}"/>
+    <!-- Gripper attachment -->
     <xacro:if value="$(arg hand)">
       <xacro:include filename="$(find franka_description)/robots/common/franka_hand.xacro"/>
@@ -32,4 +39,5 @@
        />
     </xacro:if>
+    <!-- Normal pump attachment -->
     <xacro:if value="$(arg pump)">
       <xacro:include filename="$(find franka_description)/robots/common/franka_pump.xacro"/>
@@ -39,4 +47,17 @@
           tcp_xyz="$(arg pump_tcp_xyz)"
           tcp_rpy="$(arg pump_tcp_rpy)"
+          connected_to="$(arg arm_id)_link8"
+          safety_distance="0.03"
+          gazebo="$(arg gazebo)"
+       />
+    </xacro:if>
+    <!-- Long pump attachment -->
+    <xacro:if value="$(arg long_pump)">
+      <xacro:include filename="$(find franka_description)/robots/common/franka_long_pump.xacro"/>
+      <xacro:franka_pump
+          arm_id="$(arg arm_id)"
+          rpy="0 0 ${-pi/4}"
+          tcp_xyz="$(arg long_pump_tcp_xyz)"
+          tcp_rpy="$(arg long_pump_tcp_rpy)"
           connected_to="$(arg arm_id)_link8"
           safety_distance="0.03"
